Commit message: Update URDF, Change joint order, add joint limits

File: robot.urdf (robot description, URDF)
Before this commit: robot sassa, 13 links, 12 joints
Links:
- link body_sasm: mass 4.41913 -> 4.41197
Joints:
- joint FL0: child helbow_sasm_3 -> helbow_sasm; limit effort=1 velocity=20 -> lower=-0.785398 upper=0.785398 effort=1 velocity=20; origin xyz=-0.06 0.161 -0.045 rpy=1.5708 -1.5708 0 -> xyz=-0.06 0.161 3.1225e-17 rpy=1.5708 -1.5708 0
- joint FL1: child upperleg_sasm_3 -> upperleg_sasm; limit effort=1 velocity=20 -> lower=-1.5708 upper=1.5708 effort=1 velocity=20; origin xyz=-4.16334e-17 0.016 -0.06 rpy=-1.5708 -7.45474e-28 -3.14159 -> xyz=-3.1225e-17 0.016 -0.06 rpy=-1.5708 -7.45474e-28 -3.14159; parent helbow_sasm_3 -> helbow_sasm
- joint FL2: child lowerleg_sasm_3 -> lowerleg_sasm; limit effort=1 velocity=20 -> lower=-2.35619 upper=2.35619 effort=1 velocity=20; origin xyz=0.213 6.38378e-15 -0.0685 rpy=5.37991e-16 -1.05958e-15 -1.46765e-27 -> xyz=0.213 6.43929e-15 -0.0685 rpy=5.37991e-16 -1.05958e-15 -1.46765e-27; parent upperleg_sasm_3 -> upperleg_sasm
- joint FR0: child helbow_sasm_4 -> helbow_sasm_2; limit effort=1 velocity=20 -> lower=-0.785398 upper=0.785398 effort=1 velocity=20; origin xyz=0.06 0.161 -0.045 rpy=1.5708 1.5708 0 -> xyz=0.06 0.161 3.81639e-17 rpy=1.5708 1.5708 0
- joint FR1: child upperleg_sasm_4 -> upperleg_sasm_2; limit effort=1 velocity=20 -> lower=-1.5708 upper=1.5708 effort=1 velocity=20; origin xyz=-2.08167e-17 0.016 -0.06 rpy=1.5708 -1.22125e-15 -2.75717e-16 -> xyz=-3.83799e-17 0.016 -0.06 rpy=1.5708 -1.22125e-15 -2.75717e-16; parent helbow_sasm_4 -> helbow_sasm_2
- joint FR2: child lowerleg_sasm_4 -> lowerleg_sasm_2; limit effort=1 velocity=20 -> lower=-2.35619 upper=2.35619 effort=1 velocity=20; origin xyz=0.213 5.10703e-15 -0.0685 rpy=-3.14159 6.7904e-16 -7.25635e-15 -> xyz=0.213 5.02376e-15 -0.0685 rpy=-3.14159 6.7904e-16 -7.25635e-15; parent upperleg_sasm_4 -> upperleg_sasm_2
- joint HL0: child helbow_sasm -> helbow_sasm_3; limit effort=1 velocity=20 -> lower=-0.785398 upper=0.785398 effort=1 velocity=20; origin xyz=-0.06 -0.161 -0.045 rpy=-1.5708 1.5708 0 -> xyz=-0.06 -0.161 -1.75833e-16 rpy=-1.5708 1.5708 0
- joint HL1: child upperleg_sasm -> upperleg_sasm_3; limit effort=1 velocity=20 -> lower=-1.5708 upper=1.5708 effort=1 velocity=20; origin xyz=-2.77556e-17 0.016 -0.06 rpy=1.5708 -4.94049e-14 -6.67641e-16 -> xyz=-2.93932e-17 0.016 -0.06 rpy=1.5708 -5.01088e-14 3.33067e-16; parent helbow_sasm -> helbow_sasm_3
- joint HL2: child lowerleg_sasm -> lowerleg_sasm_3; limit effort=1 velocity=20 -> lower=-2.35619 upper=2.35619 effort=1 velocity=20; origin xyz=0.213 6.77236e-15 -0.0685 rpy=2.22045e-16 -2.22045e-16 -5.76478e-15 -> xyz=0.213 7.63278e-15 -0.0685 rpy=2.81945e-15 1.54819e-14 6.71612e-15; parent upperleg_sasm -> upperleg_sasm_3
- joint HR0: child helbow_sasm_2 -> helbow_sasm_4; limit effort=1 velocity=20 -> lower=-0.785398 upper=0.785398 effort=1 velocity=20; origin xyz=0.06 -0.161 -0.045 rpy=-1.5708 -1.5708 0 -> xyz=0.06 -0.161 -1.7028e-16 rpy=-1.5708 -1.5708 0
- joint HR1: child upperleg_sasm_2 -> upperleg_sasm_4; limit effort=1 velocity=20 -> lower=-1.5708 upper=1.5708 effort=1 velocity=20; origin xyz=-2.77556e-17 0.016 -0.06 rpy=-1.5708 3.05311e-15 3.14159 -> xyz=3.27902e-18 0.016 -0.06 rpy=-1.5708 3.05311e-15 3.14159; parent helbow_sasm_2 -> helbow_sasm_4
- joint HR2: child lowerleg_sasm_2 -> lowerleg_sasm_4; limit effort=1 velocity=20 -> lower=-2.35619 upper=2.35619 effort=1 velocity=20; origin xyz=0.213 3.66374e-15 -0.0685 rpy=3.8335e-15 -2.1387e-15 -1.78641e-14 -> xyz=0.213 3.63598e-15 -0.0685 rpy=3.8335e-15 -2.1387e-15 -1.78641e-14; parent upperleg_sasm_2 -> upperleg_sasm_4

Commit message: update urdf, add a script to generate obj mesh

File: robot.urdf (robot description, URDF)
Before this commit: robot sassa, 13 links, 12 joints
Links:
- link body_sasm: mass 4.41197 -> 4.41833
Joints:
- joint FL0: origin xyz=-0.06 0.161 3.1225e-17 rpy=1.5708 -1.5708 0 -> xyz=0.161 0.06 4.03787e-17 rpy=-3.12787e-30 -1.5708 0
- joint FL1: origin xyz=-3.1225e-17 0.016 -0.06 rpy=-1.5708 -7.45474e-28 -3.14159 -> xyz=-3.06858e-17 0.016 -0.06 rpy=-1.5708 -1.40252e-27 -3.14159
- joint FL2: origin xyz=0.213 6.43929e-15 -0.0685 rpy=5.37991e-16 -1.05958e-15 -1.46765e-27 -> xyz=0.213 6.41154e-15 -0.0685 rpy=5.37991e-16 -2.21964e-15 -1.16006e-15
- joint FR0: origin xyz=0.06 0.161 3.81639e-17 rpy=1.5708 1.5708 0 -> xyz=0.161 -0.06 4.03787e-17 rpy=-3.14159 1.5708 0
- joint FR1: origin xyz=-3.83799e-17 0.016 -0.06 rpy=1.5708 -1.22125e-15 -2.75717e-16 -> xyz=-4.03316e-17 0.016 -0.06 rpy=1.5708 -1.84678e-15 3.8968e-17
- joint FR2: origin xyz=0.213 5.02376e-15 -0.0685 rpy=-3.14159 6.7904e-16 -7.25635e-15 -> xyz=0.213 5.35683e-15 -0.0685 rpy=-3.14159 7.90062e-16 -9.00322e-15
- joint HL0: origin xyz=-0.06 -0.161 -1.75833e-16 rpy=-1.5708 1.5708 0 -> xyz=-0.161 0.06 -1.7453e-16 rpy=-4.67137e-30 1.5708 0
- joint HL1: origin xyz=-2.93932e-17 0.016 -0.06 rpy=1.5708 -5.01088e-14 3.33067e-16 -> xyz=3.01347e-18 0.016 -0.06 rpy=1.5708 2.27474e-15 3.22092e-15
- joint HL2: origin xyz=0.213 7.63278e-15 -0.0685 rpy=2.81945e-15 1.54819e-14 6.71612e-15 -> xyz=0.213 7.27196e-15 -0.0685 rpy=2.22045e-16 -2.55409e-14 6.4386e-14
- joint HR0: origin xyz=0.06 -0.161 -1.7028e-16 rpy=-1.5708 -1.5708 0 -> xyz=-0.161 -0.06 -1.7453e-16 rpy=-3.14159 -1.5708 0
- joint HR1: origin xyz=3.27902e-18 0.016 -0.06 rpy=-1.5708 3.05311e-15 3.14159 -> xyz=-3.06858e-17 0.016 -0.06 rpy=-1.5708 7.32747e-15 -3.14159
- joint HR2: origin xyz=0.213 3.63598e-15 -0.0685 rpy=3.8335e-15 -2.1387e-15 -1.78641e-14 -> xyz=0.213 6.46705e-15 -0.0685 rpy=1.11022e-16 -6.12323e-17 4.4631e-14

Commit message: update max speed and torque values

File: robot.urdf (robot description, URDF)
Before this commit: robot sassa, 13 links, 12 joints
Joints:
- joint FL0: limit lower=-0.785398 upper=0.785398 effort=1 velocity=20 -> lower=-0.785398 upper=0.785398 effort=9 velocity=15
- joint FL1: limit lower=-1.5708 upper=1.5708 effort=1 velocity=20 -> lower=-1.5708 upper=1.5708 effort=9 velocity=15
- joint FL2: limit lower=-2.35619 upper=2.35619 effort=1 velocity=20 -> lower=-2.35619 upper=2.35619 effort=9 velocity=15
- joint FR0: limit lower=-0.785398 upper=0.785398 effort=1 velocity=20 -> lower=-0.785398 upper=0.785398 effort=9 velocity=15
- joint FR1: limit lower=-1.5708 upper=1.5708 effort=1 velocity=20 -> lower=-1.5708 upper=1.5708 effort=9 velocity=15
- joint FR2: limit lower=-2.35619 upper=2.35619 effort=1 velocity=20 -> lower=-2.35619 upper=2.35619 effort=9 velocity=15
- joint HL0: limit lower=-0.785398 upper=0.785398 effort=1 velocity=20 -> lower=-0.785398 upper=0.785398 effort=9 velocity=15
- joint HL1: limit lower=-1.5708 upper=1.5708 effort=1 velocity=20 -> lower=-1.5708 upper=1.5708 effort=9 velocity=15
- joint HL2: limit lower=-2.35619 upper=2.35619 effort=1 velocity=20 -> lower=-2.35619 upper=2.35619 effort=9 velocity=15
- joint HR0: limit lower=-0.785398 upper=0.785398 effort=1 velocity=20 -> lower=-0.785398 upper=0.785398 effort=9 velocity=15
- joint HR1: limit lower=-1.5708 upper=1.5708 effort=1 velocity=20 -> lower=-1.5708 upper=1.5708 effort=9 velocity=15
- joint HR2: limit lower=-2.35619 upper=2.35619 effort=1 velocity=20 -> lower=-2.35619 upper=2.35619 effort=9 velocity=15

Commit message: Add foot frame, change dof axis direction

File: robot.urdf (robot description, URDF)
Before this commit: robot sassa, 13 links, 12 joints
Links:
- added link FL_foot, mass 1e-9
- added link FR_foot, mass 1e-9
- added link HL_foot, mass 1e-9
- added link HR_foot, mass 1e-9
- link body_sasm: mass 4.41833 -> 3.4790000000000000924
- link helbow_sasm: mass 1.00534 -> 0.76500000000000001332
- link helbow_sasm_2: mass 1.00534 -> 0.76500000000000001332
- link helbow_sasm_3: mass 1.00534 -> 0.76500000000000001332
- link helbow_sasm_4: mass 1.00534 -> 0.76500000000000001332
- link lowerleg_sasm: mass 0.171662 -> 0.13200000000000006173
- link lowerleg_sasm_2: mass 0.171662 -> 0.13200000000000006173
- link lowerleg_sasm_3: mass 0.171662 -> 0.13200000000000006173
- link lowerleg_sasm_4: mass 0.171662 -> 0.13200000000000006173
- link upperleg_sasm: mass 1.09837 -> 0.90300000000000013589
- link upperleg_sasm_2: mass 1.09837 -> 0.90300000000000002487
- link upperleg_sasm_3: mass 1.09837 -> 0.90300000000000013589
- link upperleg_sasm_4: mass 1.09837 -> 0.90300000000000013589
Joints:
- added joint FL_foot_frame: type fixed, parent lowerleg_sasm, child FL_foot, origin xyz=0.21732050807564642914 -2.7339241981394479808e-14 -2.7755575615628913511e-17 rpy=-1.5707963267948950037 2.5827259566927519308e-15 1.570796326794896558, axis 0 0 0
- added joint FR_foot_frame: type fixed, parent lowerleg_sasm_2, child FR_foot, origin xyz=0.21732050807564631811 -2.7311486405778850894e-14 0 rpy=-1.5707963267948970021 8.9544612897454717878e-16 1.5707963267949038855, axis 0 0 0
- added joint HL_foot_frame: type fixed, parent lowerleg_sasm_3, child HL_foot, origin xyz=0.21732050807564634587 -2.7339241981394479808e-14 -5.5511151231257827021e-17 rpy=-1.57079632679489678 -2.7224149397708416402e-14 1.5707963267948661379, axis 0 0 0
- added joint HR_foot_frame: type fixed, parent lowerleg_sasm_4, child HR_foot, origin xyz=0.21732050807564637362 2.7283730830163221981e-14 0 rpy=-1.570796326794896558 2.2204460492510886297e-16 1.57079632679489678, axis 0 0 0
- joint FL0: limit lower=-0.785398 upper=0.785398 effort=9 velocity=15 -> lower=-0.785398163397448279 upper=0.785398163397448279 effort=9 velocity=20; origin xyz=0.161 0.06 4.03787e-17 rpy=-3.12787e-30 -1.5708 0 -> xyz=0.16100000000000047606 0.060000000000000004718 6.00732341963438899e-17 rpy=-3.1278740296522731543e-30 -1.570796326794896336 0
- joint FL1: limit lower=-1.5708 upper=1.5708 effort=9 velocity=15 -> lower=-1.570796326794896558 upper=1.570796326794896558 effort=9 velocity=20; origin xyz=-3.06858e-17 0.016 -0.06 rpy=-1.5708 -1.40252e-27 -3.14159 -> xyz=-2.1926730353241371394e-17 0.016000000000000007272 -0.05999999999999999778 rpy=-1.570796326794896558 -1.4025207337730963138e-27 -3.141592653589793116
- joint FL2: limit lower=-2.35619 upper=2.35619 effort=9 velocity=15 -> lower=-2.356194490192344837 upper=2.356194490192344837 effort=9 velocity=20; origin xyz=0.213 6.41154e-15 -0.0685 rpy=5.37991e-16 -2.21964e-15 -1.16006e-15 -> xyz=0.21300000000000002265 6.4392935428259079345e-15 -0.068500000000000116351 rpy=5.3799142389700426073e-16 -2.219643924176522297e-15 -1.160061430643682592e-15
- joint FR0: limit lower=-0.785398 upper=0.785398 effort=9 velocity=15 -> lower=-0.785398163397448279 upper=0.785398163397448279 effort=9 velocity=20; origin xyz=0.161 -0.06 4.03787e-17 rpy=-3.14159 1.5708 0 -> xyz=0.16100000000000047606 -0.059999999999999990841 5.6159486713100279927e-17 rpy=-3.141592653589793116 1.570796326794896336 0
- joint FR1: limit lower=-1.5708 upper=1.5708 effort=9 velocity=15 -> lower=-1.570796326794896558 upper=1.570796326794896558 effort=9 velocity=20; origin xyz=-4.03316e-17 0.016 -0.06 rpy=1.5708 -1.84678e-15 3.8968e-17 -> xyz=-4.2430336288061214674e-17 0.015999999999999993394 -0.05999999999999999778 rpy=-1.57079632679489678 -1.8467845446348508561e-15 3.896800864265682098e-17
- joint FR2: limit lower=-2.35619 upper=2.35619 effort=9 velocity=15 -> lower=-2.356194490192344837 upper=2.356194490192344837 effort=9 velocity=20; origin xyz=0.213 5.35683e-15 -0.0685 rpy=-3.14159 7.90062e-16 -9.00322e-15 -> xyz=0.21300000000000654521 -5.3568260938163803075e-15 0.06850000000000018574 rpy=6.9248076212676153043e-15 -7.9006181994192093522e-16 9.0032171146696425232e-15
- joint HL0: limit lower=-0.785398 upper=0.785398 effort=9 velocity=15 -> lower=-0.785398163397448279 upper=0.785398163397448279 effort=9 velocity=20; origin xyz=-0.161 0.06 -1.7453e-16 rpy=-4.67137e-30 1.5708 0 -> xyz=-0.16099999999999917155 0.060000000000000011657 -1.9408453586391257677e-16 rpy=-4.6713694273552509586e-30 1.570796326794896558 0
- joint HL1: limit lower=-1.5708 upper=1.5708 effort=9 velocity=15 -> lower=-1.570796326794896558 upper=1.570796326794896558 effort=9 velocity=20; origin xyz=3.01347e-18 0.016 -0.06 rpy=1.5708 2.27474e-15 3.22092e-15 -> xyz=-3.0418668761338497323e-17 0.015999999999999986455 -0.05999999999999999778 rpy=1.570796326794896558 2.2747394953037020346e-15 3.2209162361520329144e-15
- joint HL2: limit lower=-2.35619 upper=2.35619 effort=9 velocity=15 -> lower=-2.356194490192344837 upper=2.356194490192344837 effort=9 velocity=20; origin xyz=0.213 7.27196e-15 -0.0685 rpy=2.22045e-16 -2.55409e-14 6.4386e-14 -> xyz=0.21300000000000055 7.2719608112947753398e-15 -0.06849999999999886735 rpy=2.2204460491921242353e-16 -2.5540850755104416721e-14 6.4385996534355664365e-14
- joint HR0: limit lower=-0.785398 upper=0.785398 effort=9 velocity=15 -> lower=-0.785398163397448279 upper=0.785398163397448279 effort=9 velocity=20; origin xyz=-0.161 -0.06 -1.7453e-16 rpy=-3.14159 -1.5708 0 -> xyz=-0.16099999999999917155 -0.059999999999999983902 -1.9781398741257412101e-16 rpy=-3.141592653589793116 -1.5707963267947993025 0
- joint HR1: limit lower=-1.5708 upper=1.5708 effort=9 velocity=15 -> lower=-1.570796326794896558 upper=1.570796326794896558 effort=9 velocity=20; origin xyz=-3.06858e-17 0.016 -0.06 rpy=-1.5708 7.32747e-15 -3.14159 -> xyz=-3.6033927686494999687e-17 0.016000000000000305644 -0.05999999999999999778 rpy=1.570796326794896558 7.3274719625260410554e-15 -3.141592653589793116
- joint HR2: limit lower=-2.35619 upper=2.35619 effort=9 velocity=15 -> lower=-2.356194490192344837 upper=2.356194490192344837 effort=9 velocity=20; origin xyz=0.213 6.46705e-15 -0.0685 rpy=1.11022e-16 -6.12323e-17 4.4631e-14 -> xyz=0.21300000000000002265 -6.467049118441536848e-15 0.068499999999999963696 rpy=1.1102230246387924942e-16 6.1232339957382020092e-17 -4.4630965589931286614e-14
